Commit message: improved zerg urdf, corrected topics in launch files

File: gki_zerg_description/robots/zerg.urdf.xacro (robot description, xacro)
@@ -8,4 +8,5 @@
   <xacro:include filename="$(find gki_sensors_description)/urdf/hokuyo_urg.urdf.xacro" />
   <xacro:include filename="$(find gki_sensors_description)/urdf/sick_rfu620.urdf.xacro" />
+  <xacro:include filename="$(find gki_sensors_description)/urdf/xsens_imu.urdf.xacro" />
   <xacro:include filename="$(find gki_cube_gripper_description)/urdf/cube_gripper.urdf.xacro" />
   <!--
@@ -36,4 +37,10 @@
 			<origin xyz="0.23 0.0 0.0625" rpy="0 0 0"/>
 		</item_bar_40_20>
+		<item_bar_20_20 name="gripper_attach_right_bar" parent="${parent}" length="0.08">
+			<origin xyz="0.19 -0.1 0.11" rpy="0 ${90*M_DEGREES} 0"/>
+		</item_bar_20_20>
+		<item_bar_20_20 name="gripper_attach_left_bar" parent="${parent}" length="0.08">
+			<origin xyz="0.19 0.1 0.11" rpy="0 ${90*M_DEGREES} 0"/>
+		</item_bar_20_20>
 	</xacro:macro>
   <zerg_base/>
@@ -43,24 +50,13 @@
   </xacro:hokuyo_urg>
 	<xacro:sick_rfu620 name="rfid_sensor" parent="base_link" ros_topic="rfid_tag">
-		<origin xyz="-0.235 0.0 0.325" rpy="0 3.1415 0"/>
+		<origin xyz="-0.235 0.0 0.325" rpy="0 ${180*M_DEGREES} 0"/>
 	</xacro:sick_rfu620>
+	<xacro:xsens_imu name="imu" parent="base_link">
+		<origin xyz="-0.215 0.0 0.345" rpy="0 0 0"/>
+	</xacro:xsens_imu>
 	<xacro:cube_gripper name="cube_gripper" parent="base_link">
-		<origin xyz="0.235 0.0 0.325" rpy="0 0 0"/>
+		<origin xyz="0.2 0.0 0.11" rpy="${180*M_DEGREES} 0 0"/>
 	</xacro:cube_gripper>
 	<!--
-  <joint name="imu_joint" type="fixed">
-      <origin xyz="0.056 0.062 0.0202" rpy="0 0 0"/>
-      <parent link="base_link"/>
-      <child link="imu_link"/>
-  </joint>
-  <link name="imu_link">
-      <inertial>
-          <mass value="0.001"/>
-          <origin xyz="0 0 0" rpy="0 0 0"/>
-          <inertia ixx="0.0001" ixy="0" ixz="0"
-              iyy="0.000001" iyz="0"
-              izz="0.0001"/>
-      </inertial>
-  </link>
 -->
 </robot>

Commit message: parameter tuning

File: gki_zerg_description/robots/zerg.urdf.xacro (robot description, xacro)
@@ -34,5 +34,5 @@
 			<origin xyz="0.19 0.0 0.0625" rpy="0 0 ${90*M_DEGREES}"/>
 		</item_bar_20_20>
-		<item_bar_40_20 name="front_tip_bar" parent="${parent}" length="0.065">
+		<item_bar_40_20 name="front_tip_bar" parent="${parent}" length="0.15">
 			<origin xyz="0.23 0.0 0.0625" rpy="0 0 0"/>
 		</item_bar_40_20>
@@ -47,5 +47,5 @@
 	<sickrd_2016_parts parent="base_link"/>
   <xacro:hokuyo_urg name="base_laser" parent="base_link" ros_topic="base_scan" update_rate="30" ray_count="1080" min_angle="135" max_angle="-135">
-    <origin xyz="0.215 0.0 0.08" rpy="0 0 0"/>
+    <origin xyz="0.275 0.0 0.08" rpy="0 0 0"/>
   </xacro:hokuyo_urg>
 	<xacro:sick_rfu620 name="rfid_sensor" parent="base_link" ros_topic="rfid_tag">
